File: Schematic/GasHeaterControl/GasHeaterControl.kicad_sch (KiCad schematic)
At the start: 6 parts, among them K1 Finder 46.61.9.024.0040, P0 Conn_WallPlug_Earth, SW0 SW_SPDT

Commit message: updates on README and the schematics
Parts:
- renumbered R12 to R1
Other:
- note added: "Arduino Mega"
- note removed: "Arduino Uno"
Changed lines of the file:
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@@
     (effects (font (size 1.27 1.27)) (justify left bottom))
   )
-  (text "Arduino Uno" (at 168.91 63.5 0)
+  (text "Arduino Mega" (at 168.91 63.5 0)
     (effects (font (size 2 2)) (justify left bottom))
   )
@@
   (symbol (lib_id "Device:Heater") (at 242.57 110.49 270) (unit 1)
     (in_bom yes) (on_board yes)
-    (property "Reference" "R12" (id 0) (at 242.57 105.2322 90))
+    (property "Reference" "R1" (id 0) (at 242.57 105.2322 90))
     (property "Value" "Heater" (id 1) (at 242.57 107.5436 90))
     (property "Footprint" "" (id 2) (at 242.57 108.712 90)
